Commit message: add RH-P12-RN-A support to MoveIt config

File: ur_moveit_config/srdf/ur_macro.srdf.xacro (robot description, xacro)
@@ -12,5 +12,8 @@
     <!--SUBGROUPS - Groups can also be formed by referencing to already defined group names-->
     <group name="ur_manipulator">
-      <chain base_link="base_link" tip_link="tool0" />
+      <chain base_link="base_link" tip_link="end_effector_link" />
+    </group>
+    <group name="gripper">
+        <joint name="rh_r1_joint"/>
     </group>
     <!--GROUP STATES - Purpose - Define a named state for a particular group, in terms of joint values. This is useful to define states like 'folded arms'-->
@@ -39,4 +42,10 @@
       <joint name="wrist_3_joint" value="-0.11" />
     </group_state>
+    <group_state name="open" group="gripper">
+        <joint name="rh_r1_joint" value="0.0"/>
+    </group_state>
+    <group_state name="closed" group="gripper">
+        <joint name="rh_r1_joint" value="1.0"/>
+    </group_state>
     <!--END EFFECTOR - Purpose - Represent information about an end effector.-->
     <!--VIRTUAL JOINT - Purpose - this element defines a virtual joint between a robot link and an external frame of reference (considered fixed with respect to the robot)-->
@@ -53,4 +62,20 @@
     <disable_collisions link1="wrist_1_link" link2="wrist_3_link" reason="Never" />
     <disable_collisions link1="wrist_2_link" link2="wrist_3_link" reason="Adjacent" />
+    <!-- Disable gripper collisions -->
+    <disable_collisions link1="rh_p12_rn_l1" link2="rh_p12_rn_l2" reason="Adjacent" />
+    <disable_collisions link1="rh_p12_rn_l1" link2="rh_p12_rn_r2" reason="Adjacent" />
+    <disable_collisions link1="rh_p12_rn_l2" link2="rh_p12_rn_r2" reason="Adjacent" />
+    <disable_collisions link1="rh_p12_rn_l2" link2="rh_p12_rn_r1" reason="Adjacent" />
+    <disable_collisions link1="rh_p12_rn_l1" link2="rh_p12_rn_r1" reason="Adjacent" />
+    <disable_collisions link1="rh_p12_rn_r1" link2="rh_p12_rn_r2" reason="Adjacent" />
+    <disable_collisions link1="rh_p12_rn_base" link2="rh_p12_rn_l1" reason="Adjacent" />
+    <disable_collisions link1="rh_p12_rn_base" link2="rh_p12_rn_l2" reason="Never" />
+    <disable_collisions link1="rh_p12_rn_base" link2="rh_p12_rn_r1" reason="Adjacent" />
+    <disable_collisions link1="rh_p12_rn_base" link2="rh_p12_rn_r2" reason="Never" />
+    <disable_collisions link1="rh_p12_rn_base" link2="wrist_3_link" reason="Adjacent" />
+    <disable_collisions link1="rh_p12_rn_l1" link2="rh_p12_rn_ee" reason="Adjacent" />
+    <disable_collisions link1="rh_p12_rn_r1" link2="rh_p12_rn_ee" reason="Adjacent" />
+    <disable_collisions link1="rh_p12_rn_l2" link2="rh_p12_rn_ee" reason="Adjacent" />
+    <disable_collisions link1="rh_p12_rn_r2" link2="rh_p12_rn_ee" reason="Adjacent" />
   </xacro:macro>
 </robot>
